File: quadcopter.sch (EAGLE design)
At the start: 82 parts, among them J1 ISP, J4 2.1MMJACKTHM, U1 ATMEGA128RFA1, Y1 16MHz, Y2 32.768kHz

Commit message: Add files via upload
Board Layout
Parts:
- removed ANDREW1: LSM9DS1, Quadparts:LSM9DS1
- removed CVBATH: 1000uF, quadparts_prebuilt:CAPACITOR-POL_SMD-7043-D_TANTALUM-220UF
- removed CVBATL: 10uF, quadparts_prebuilt:CAPACITOR-POL_SMD-7043-D_TANTALUM-220UF
- removed J4: 2.1MMJACKTHM, Quad_Lab2:2.1MMJACKTHM
- removed LED2, LED3: GREEN, SparkFun-LED:LED0603
- removed R5, R6: 330, SparkFun:RESISTOR0402-RES
- removed U$6, U$8: MOSFET, Quadparts:MOSFET
- removed U$7: MOTOR_PADS, quadparts_prebuilt:MOTOR_PADS
- added D10: Orange, quadparts_prebuilt:DIODE-LED_SMD-2012-0805
- added J2: (no value), quadparts_prebuilt:MALE_HEADER_2POS-2X1-0.1IN
- added MOSFET1, MOSFET2, MOSFET3, MOSFET4: SI2302, quadparts_prebuilt:SI2302
- added R10: 330, quadparts_prebuilt:RESISTOR_SMD-2012-0805-330
- added R11: 100, quadparts_prebuilt:RESISTOR_SMD-2012-0805-100
- C3: value 1uF -> 1000uF
- C4: value 1uF -> 10uF
- U$3: value MOSFET -> MOTOR_PADS; device Quadparts:MOSFET -> quadparts_prebuilt:MOTOR_PADS
- U$5: value MOSFET -> IMULAST; device Quadparts:MOSFET -> QuadpartsUpdated:IMULAST
Connections:
- removed net N$1: SERIAL_PROGRAMMER.4
- removed net N$12: SERIAL_DEBUGGER.4
- removed net N$13: LED2.A, R6.1
- removed net N$32: C12.2, C24.2
- removed net N$8: LED3.A, R5.1
- new net N$35: D10.A, R10.1
- net 3V: now also U$5.CS_A/G, U$5.CS_M, U$5.SDO_M, U$5.VDD, U$5.VDDD; no longer ANDREW1.CS_A/G, ANDREW1.CS_M, ANDREW1.VDD, ANDREW1.VDDD
- net BAT_GND: now also C12.2, C24.2, D10.C, R11.1
- net GND: now also MOSFET1.S, MOSFET2.S, MOSFET3.S, MOSFET4.S, R11.2, U$5.GND, U$5.GNDD, U$5.RES, U$5.RESS, U$5.RESSS, U$5.RESSSS, U$5.RESSSSS; no longer ANDREW1.GND, ANDREW1.GNDD, ANDREW1.RES, ANDREW1.RESS, ANDREW1.RESSS, ANDREW1.RESSSS, ANDREW1.RESSSSS, ANDREW1.SDO_M, CVBATH.-, CVBATL.-, LED2.C, LED3.C, U$3.S, U$5.S, U$6.S, U$8.S
- net N$14: now also MOSFET1.D; no longer U$5.D
- net N$15: now also MOSFET1.G; no longer U$5.G
- net N$17: now also J2.2; no longer J4.RING, J4.RING_SW
- net N$19: now also MOSFET2.D; no longer U$3.D
- net N$2: now also U$5.VDD_IO, U$5.VDD__IO; no longer ANDREW1.VDD_IO, ANDREW1.VDD__IO
- net N$20: now also MOSFET2.G; no longer U$3.G
- net N$23: now also U$5.C1; no longer ANDREW1.C1
- net N$24: now also MOSFET3.D, U$3.V-; no longer U$4.V-, U$6.D
- net N$25: now also MOSFET3.G; no longer U$6.G
- net N$29: now also MOSFET4.D, U$4.V-; no longer U$7.V-, U$8.D
- net N$30: now also MOSFET4.G; no longer U$8.G
- net N$33: now also U$5.CAP; no longer ANDREW1.CAP
- net N$34: now also U$5.P$5; no longer ANDREW1.P$5
- net PB6: no longer R5.2
- net PB7: no longer R6.2
- net SCL: now also U$5.SCL/SPC; no longer ANDREW1.SCL/SPC
- net SDA: now also U$5.SDA/SDI/SDO; no longer ANDREW1.SDA/SDI/SDO
- net VBAT: now also J2.1, R10.2, U$3.V+; no longer CVBATH.+, CVBATL.+, J4.TIP, U$7.V+
Other:
- note removed: "ASK about the polarity and switch"
- note removed: "ask"
- moved on the sheet: U$4
