File: quadcopter.sch (EAGLE design)
At the start: 79 parts, among them J1 ISP, U1 ATMEGA128RFA1, Y1 16MHz, Y2 32.768kHz

Commit message: Fixed Schematic but still not able to root 90%
Parts:
- removed A1: ANTENNA2SMD5, SparkFun-RF:ANTENNA2SMD5
- removed B1: 748421245, SparkFun-RF:BALUN0805
- removed C24: 10nF, quadparts_prebuilt:CAPACITOR-NP_SMD-2012-0805_CERAMIC-1UF
- removed C25: 10nF, quadparts_prebuilt:CAPACITOR-NP_SMD-2012-0805_CERAMIC
- removed C26, C28: 100nF, quadparts_prebuilt:CAPACITOR-NP_SMD-2012-0805_CERAMIC
- removed C27: 10uF, quadparts_prebuilt:CAPACITOR-NP_SMD-2012-0805_CERAMIC
- removed C6: 12pF, SparkFun-Passives:CAP0402-CAP
- removed CG, CG1, CG2, CG3: 1uF, quadparts_prebuilt:CAPACITOR-NP_SMD-2012-0805_CERAMIC
- removed D10: Orange, quadparts_prebuilt:DIODE-LED_SMD-2012-0805
- removed D6: Green, quadparts_prebuilt:DIODE-LED_SMD-2012-0805
- removed R10, R2: 330, quadparts_prebuilt:RESISTOR_SMD-2012-0805-330
- removed R8: 10K, quadparts_prebuilt:RESISTOR_SMD-2012-0805-10K
- removed RG1, RG3, RG5, RG7: 100, quadparts_prebuilt:RESISTOR_SMD-2012-0805
- removed RG2, RG4, RG6, RG8: 10K, quadparts_prebuilt:RESISTOR_SMD-2012-0805
- removed U1: ATMEGA128RFA1, SparkFun-DigitalIC:ATMEGA128RFA1
- removed Y1: 16MHz, SparkFun-FreqCtrl:CRYSTAL5X3
- added ANDREW1: LSM9DS1, QuadpartsUpdated:LSM9DS1
- added B2: BALUN0805, quadparts_prebuilt:BALUN0805
- added C13, C14, C18: 1uF, quadparts_prebuilt:CAPACITOR-NP_SMD-2012-0805_CERAMIC-1UF
- added C19, C20: 0.1uF, quadparts_prebuilt:CAPACITOR-NP_SMD-2012-0805_CERAMIC-0.1UF
- added C21: 0.01uF, quadparts_prebuilt:CAPACITOR-NP_SMD-2012-0805_CERAMIC-0.01UF
- added J7, M1, M2, M3, M4: (no value), quadparts_prebuilt:MALE_HEADER_2POS-2X1-0.1IN
- added R12, R14, R16, R18: 100, quadparts_prebuilt:RESISTOR_SMD-2012-0805-100
- added R13, R15, R17, R5, R6: 10K, quadparts_prebuilt:RESISTOR_SMD-2012-0805-10K
- added U2: ATMEGA128RFA1, quadparts_prebuilt:ATMEGA128RFA1
- C1, C2: value 1uF -> 12pF; device SparkFun-Passives:CAP0402-CAP -> quadparts_prebuilt:CAPACITOR-NP_SMD-2012-0805_CERAMIC-12PF
- C10: value 100nF -> 1uF; device quadparts_prebuilt:CAPACITOR-NP_SMD-2012-0805_CERAMIC -> quadparts_prebuilt:CAPACITOR-NP_SMD-2012-0805_CERAMIC-1UF
- C11: value 22pF -> 1uF; device SparkFun-Passives:CAP0402-CAP -> quadparts_prebuilt:CAPACITOR-NP_SMD-2012-0805_CERAMIC-1UF
- C12: value 10uF -> 1uF
- C15: device SparkFun-Passives:CAP0402-CAP -> quadparts_prebuilt:CAPACITOR-NP_SMD-2012-0805_CERAMIC-0.1UF
- C16: value JUMP -> 1uF; device SparkFun:CAP0402-CAP -> quadparts_prebuilt:CAPACITOR-NP_SMD-2012-0805_CERAMIC-1UF
- C17: value JUMP -> 10uF; device SparkFun:CAP0402-CAP -> quadparts_prebuilt:CAPACITOR-NP_SMD-2012-0805_CERAMIC-10UF
- C22: value 1uF -> 22pF; device quadparts_prebuilt:CAPACITOR-NP_SMD-2012-0805_CERAMIC-1UF -> quadparts_prebuilt:CAPACITOR-NP_SMD-2012-0805_CERAMIC-22PF
- C3: value 1000uF -> 1uF; device SparkFun-Passives:CAP0402-CAP -> quadparts_prebuilt:CAPACITOR-NP_SMD-2012-0805_CERAMIC-1UF
- C4: device SparkFun-Passives:CAP0402-CAP -> quadparts_prebuilt:CAPACITOR-NP_SMD-2012-0805_CERAMIC-10UF
- C5: value 12pF -> 220uF; device SparkFun-Passives:CAP0402-CAP -> quadparts_prebuilt:CAPACITOR-POL_SMD-7043-D_TANTALUM-220UF
- C7: value 12pF -> 10uF; device SparkFun-Passives:CAP0402-CAP -> quadparts_prebuilt:CAPACITOR-NP_SMD-2012-0805_CERAMIC-10UF
- C8: value 12pF -> 0.01uF; device SparkFun-Passives:CAP0402-CAP -> quadparts_prebuilt:CAPACITOR-NP_SMD-2012-0805_CERAMIC-0.01UF
- C9: device SparkFun-Passives:CAP0402-CAP -> quadparts_prebuilt:CAPACITOR-NP_SMD-2012-0805_CERAMIC-0.75PF
- R1: value 10k -> 10K; device SparkFun-Passives:RESISTOR0402-RES -> quadparts_prebuilt:RESISTOR_SMD-2012-0805-10K
- R11: value 100 -> 10K; device quadparts_prebuilt:RESISTOR_SMD-2012-0805-100 -> quadparts_prebuilt:RESISTOR_SMD-2012-0805-10K
- U$5: value IMULAST -> ANTENNA2SMD5; device QuadpartsUpdated:IMULAST -> quadparts_prebuilt:ANTENNA2SMD5
- Y2: value 32.768kHz -> (none); device SparkFun-FreqCtrl:CRYSTAL32-SMD -> quadparts_prebuilt:CRYSTAL5X3
Connections:
- removed net A0: U1.PF0(ADC0)
- removed net N$10: B1.OUT1, C16.2
- removed net N$11: B1.OUT2, C17.1
- removed net N$25: MOSFET3.G, RG5.1, RG6.1
- removed net N$30: MOSFET4.G, RG7.1, RG8.1
- removed net N$31: D6.A, R2.1
- removed net N$34: R8.2, U$5.P$5
- removed net N$35: D10.A, R10.1
- removed net N$5: C7.1, U1.PG4(TOSC1), Y2.1
- removed net N$6: C8.1, U1.PG3(TOSC2), Y2.2
- removed net PG5: U1.PG5(OC0B)
- removed net TST: U1.TST
- new net N$48: MOSFET2.G
- new net N$50: MOSFET3.G
- new net N$52: C18.1, MOSFET4.G, R17.2, R18.2
- new net VBAT_SENSE: R5.1, R6.2, U2.PF0(ADC0)
- net 3V: now also ANDREW1.CS_A/G, ANDREW1.CS_M, ANDREW1.DEN_A/G, ANDREW1.SDO_A/G, ANDREW1.SDO_M, ANDREW1.VDD1, ANDREW1.VDD2, ANDREW1.VDD_IO, ANDREW1.VDD__IO, C16.1, C17.2, C19.2, J7.1, U2.DEVDD, U2.EVDD; no longer C23.1, C26.2, C27.2, R8.1, U$5.CS_A/G, U$5.CS_M, U$5.SDO_M, U$5.VDD, U$5.VDDD, U1.DEVDD, U1.EVDD
- net A1: now also U2.PF1(ADC1); no longer U1.PF1(ADC1)
- net A2: now also U2.PF2(ADC2/DIG2); no longer U1.PF2(ADC2/DIG2)
- net A3: now also U2.PF3(ADC3/DIG4); no longer U1.PF3(ADC3/DIG4)
- net A4: now also U2.PF4(ADC4/TCK); no longer U1.PF4(ADC4/TCK)
- net A5: now also U2.PF5(ADC5/TMS); no longer U1.PF5(ADC5/TMS)
- net A6: now also U2.PF6(ADC6/TDO); no longer U1.PF6(ADC6/TDO)
- net A7: now also U2.PF7(ADC7/TDI); no longer U1.PF7(ADC7/TDI)
- net AREF: now also U2.AREF; no longer U1.AREF
- net AVDD: now also C11.1, U2.AVDD; no longer C1.1, U1.AVDD
- net BAT_GND: now also C5.-, C7.2, C8.2; no longer C12.2, C24.2, D10.C, D6.C, R11.1
- net DVDD: now also C23.1, U2.DVDD; no longer C2.1, U1.DVDD
- net GND: now also ANDREW1.GND1, ANDREW1.GND2, ANDREW1.RES1, ANDREW1.RES2, ANDREW1.RES3, ANDREW1.RES4, ANDREW1.RES5, B2.GND@5, C12.2, C13.2, C14.2, C16.2, C17.1, C18.2, C19.1, C20.1, C21.2, C22.1, C9.2, J7.2, M1.1, M2.1, M3.1, M4.1, R11.1, R13.1, R15.1, R17.1, R6.1, U2.AVSS, U2.AVSS_RFN, U2.AVSS_RFP, U2.CLKI, U2.DVSS, U2.TST; no longer B1.GND@5, C22.2, C25.2, C26.1, C27.1, C28.1, C5.2, C6.2, C7.2, C8.2, C9.1, CG.2, CG1.2, CG2.2, CG3.2, R11.2, RG2.2, RG4.2, RG6.2, RG8.2, U$5.GND, U$5.GNDD, U$5.RES, U$5.RESS, U$5.RESSS, U$5.RESSSS, U$5.RESSSSS, U1.AVSS, U1.AVSS_RFN, U1.AVSS_RFP, U1.CLKI, U1.DVSS, U1.PADDLE
- net MISO: now also U2.PB3(MISO/PDO/PCINT3); no longer U1.PB3(MISO/PDO/PCINT3)
- net MOSI: now also U2.PB2(MOSI/PDI/PCINT2); no longer U1.PB2(MOSI/PDI/PCINT2)
- net N$15: now also C13.1, R13.2, R14.2; no longer MOSFET1.G, RG1.1, RG2.1
- net N$2: now also MOSFET1.G, R11.2, R12.2; no longer U$5.VDD_IO, U$5.VDD__IO
- net N$20: now also C14.1, R15.2, R16.2; no longer MOSFET2.G, RG3.1, RG4.1
- net N$23: now also ANDREW1.C1, C20.2; no longer C28.2, U$5.C1
- net N$26: now also C12.1; no longer C22.1
- net N$3: now also C2.1, U2.XTAL1, Y2.2; no longer C5.1, U1.XTAL1, Y1.2
- net N$33: now also ANDREW1.CAP, C21.1; no longer C25.1, U$5.CAP
- net N$4: now also C1.1, U2.XTAL2, Y2.1; no longer C6.1, U1.XTAL2, Y1.1
- net N$7: now also B2.GND@2, C22.2; no longer B1.GND@2, C11.1
- net PB4: now also U2.PB4(OC2A/PCINT4); no longer U1.PB4(OC2A/PCINT4)
- net PB6: now also U2.PB6(OC1B/PCINT6); no longer U1.PB6(OC1B/PCINT6)
- net PB7: now also U2.PB7(OC0A/OC1C/PCINT7); no longer U1.PB7(OC0A/OC1C/PCINT7)
- net PD4: now also U2.PD4(ICP1); no longer U1.PD4(ICP1)
- net PD5: now also U2.PD5(XCK1); no longer U1.PD5(XCK1)
- net PD6: now also U2.PD6(T1); no longer U1.PD6(T1)
- net PD7: now also U2.PD7(T0); no longer U1.PD7(T0)
- net PE2: now also U2.PE2(XCK0/AIN0); no longer U1.PE2(XCK0/AIN0)
- net PE6: now also U2.PE6(T3/INT6); no longer U1.PE6(T3/INT6)
- net PE7: now also U2.PE7(ICP3/INT7/CLKO); no longer U1.PE7(ICP3/INT7/CLKO)
- net PG0: now also U2.PG0(DIG3); no longer U1.PG0(DIG3)
- net PG1: now also U2.PG1(DIG1); no longer U1.PG1(DIG1)
- net PG2: now also U2.PG2(AMR); no longer U1.PG2(AMR)
- net PWM1: now also M1.2, R12.1, U2.PB5(OC1A/PCINT5); no longer CG.1, RG1.2, U1.PB5(OC1A/PCINT5)
- net PWM2: now also M2.2, R14.1, U2.PE5(OC3C/INT5); no longer CG1.1, RG3.2, U1.PE5(OC3C/INT5)
- net PWM3: now also M3.2, R16.1, U2.PE3(OC3A/AIN1); no longer CG2.1, RG5.2, U1.PE3(OC3A/AIN1)
- net PWM4: now also M4.2, R18.1, U2.PE4(OC3B/INT4); no longer CG3.1, RG7.2, U1.PE4(OC3B/INT4)
- net RESET: now also U2.RSTN; no longer U1.RSTN
- net RFANT: now also B2.IN, C9.1, U$5.SIGNAL; no longer A1.SIGNAL, B1.IN, C9.2
- net RFN: now also B2.OUT2, U2.RFN; no longer C17.2, U1.RFN
- net RFP: now also B2.OUT1, U2.RFP; no longer C16.1, U1.RFP
- net RSTON: now also U2.RSTON; no longer U1.RSTON
- net RX0: now also SERIAL_PROGRAMMER.3, U2.PE0(RXD0/PCINT8); no longer U1.PE0(RXD0/PCINT8)
- net RX1: now also U2.PD2(RXD1/INT2); no longer SERIAL_PROGRAMMER.3, U1.PD2(RXD1/INT2)
- net SCK: now also U2.PB1(SCK/PCINT1); no longer U1.PB1(SCK/PCINT1)
- net SCL: now also ANDREW1.SCL/SPC, U2.PD0(SCL/INT0); no longer U$5.SCL/SPC, U1.PD0(SCL/INT0)
- net SDA: now also ANDREW1.SDA/SDI/SDO, U2.PD1(SDA/INT1); no longer U$5.SDA/SDI/SDO, U1.PD1(SDA/INT1)
- net SSN: now also U2.PB0(SSN/PCINT0); no longer U1.PB0(SSN/PCINT0)
- net TX0: now also SERIAL_PROGRAMMER.2, U2.PE1(TXD0); no longer U1.PE1(TXD0)
- net TX1: now also U2.PD3(TXD1/INT3); no longer SERIAL_PROGRAMMER.2, U1.PD3(TXD1/INT3)
- net VBAT: now also C5.+, C7.1, C8.1, R5.2; no longer C12.1, C24.1, R10.2, R2.2
Other:
- moved on the sheet: C10, C12, C22, C23, D9, R11, Y2

Commit message: Route 100% FINALLY.
Parts:
- removed ANDREW1: LSM9DS1, QuadpartsUpdated:LSM9DS1
- added R2, R8: 10K, quadparts_prebuilt:RESISTOR_SMD-2012-0805-10K
- added U$6: IMULAST, QuadpartsUpdated:IMULAST
- added U$7: WIRE_BRIDGE, QuadpartsUpdated:WIRE_BRIDGE
Connections:
- removed net AREF: U2.AREF
- net 3V: now also R2.2, R8.2, U$6.CS_A/G, U$6.CS_M, U$6.DEN_A/G, U$6.SDO_A/G, U$6.SDO_M, U$6.VDD1, U$6.VDD2, U$6.VDD_IO, U$6.VDD__IO, U2.AREF; no longer ANDREW1.CS_A/G, ANDREW1.CS_M, ANDREW1.DEN_A/G, ANDREW1.SDO_A/G, ANDREW1.SDO_M, ANDREW1.VDD1, ANDREW1.VDD2, ANDREW1.VDD_IO, ANDREW1.VDD__IO
- net BAT_GND: now also U$7.GND
- net GND: now also U$6.GND1, U$6.GND2, U$6.RES1, U$6.RES2, U$6.RES3, U$6.RES4, U$6.RES5, U$7.BATT_GND; no longer ANDREW1.GND1, ANDREW1.GND2, ANDREW1.RES1, ANDREW1.RES2, ANDREW1.RES3, ANDREW1.RES4, ANDREW1.RES5
- net N$23: now also U$6.C1; no longer ANDREW1.C1
- net N$33: now also U$6.CAP; no longer ANDREW1.CAP
- net SCL: now also R8.1, U$6.SCL/SPC; no longer ANDREW1.SCL/SPC
- net SDA: now also R2.1, U$6.SDA/SDI/SDO; no longer ANDREW1.SDA/SDI/SDO

Commit message: After fixing professor's comments
Parts:
- removed C7: 10uF, quadparts_prebuilt:CAPACITOR-NP_SMD-2012-0805_CERAMIC-10UF
- removed C8: 0.01uF, quadparts_prebuilt:CAPACITOR-NP_SMD-2012-0805_CERAMIC-0.01UF
- added C6: 0.1uF, quadparts_prebuilt:CAPACITOR-NP_SMD-2012-0805_CERAMIC-0.1UF
- C10, C13, C14: value 1uF -> 0.1uF; device quadparts_prebuilt:CAPACITOR-NP_SMD-2012-0805_CERAMIC-1UF -> quadparts_prebuilt:CAPACITOR-NP_SMD-2012-0805_CERAMIC-0.1UF
- D1, D2, D3, D4: value (none) -> 360mV; device quadparts_prebuilt:DIODE-SCHOTTKY_SMD-SOD123 -> quadparts_prebuilt:DIODE-SCHOTTKY_SMD-SOD123-360MV
Connections:
- removed net N$15: C13.1, R13.2, R14.2
- removed net N$20: C14.1, R15.2, R16.2
- net BAT_GND: now also C10.2, C13.2, C14.2, C18.2, C6.2, M1.1, M2.1, M3.1, M4.1, MOSFET1.S, MOSFET2.S, MOSFET3.S, MOSFET4.S, R11.1, R13.1, R15.1, R17.1; no longer C7.2, C8.2
- net GND: no longer C10.2, C13.2, C14.2, C18.2, M1.1, M2.1, M3.1, M4.1, MOSFET1.S, MOSFET2.S, MOSFET3.S, MOSFET4.S, R11.1, R13.1, R15.1, R17.1
- net N$2: now also C13.1; no longer C10.1
- net N$48: now also C14.1, R13.2, R14.2
- net N$50: now also C10.1, R15.2, R16.2
- net N$52: now also C6.1; no longer C18.1
- net VBAT: now also C18.1; no longer C7.1, C8.1
Other:
- moved on the sheet: C10, C13, C14, C18

Commit message: After fixing professor's comments V2
Parts:
- added C24, C25, C7, C8: 220uF, quadparts_prebuilt:CAPACITOR-POL_SMD-7043-D_TANTALUM-220UF
Connections:
- net BAT_GND: now also C24.-, C25.-, C7.-, C8.-
- net VBAT: now also C24.+, C25.+, C7.+, C8.+
Changed lines of the file:
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@@
 <part name="D4" library="quadparts_prebuilt" deviceset="DIODE-SCHOTTKY_" device="SMD-SOD123-360MV" value="360mV"/>
 <part name="C18" library="quadparts_prebuilt" deviceset="CAPACITOR-NP_" device="SMD-2012-0805_CERAMIC-1UF" value="1uF"/>
+<part name="C7" library="quadparts_prebuilt" deviceset="CAPACITOR-POL_" device="SMD-7043-D_TANTALUM-220UF" value="220uF"/>
+<part name="C8" library="quadparts_prebuilt" deviceset="CAPACITOR-POL_" device="SMD-7043-D_TANTALUM-220UF" value="220uF"/>
+<part name="C24" library="quadparts_prebuilt" deviceset="CAPACITOR-POL_" device="SMD-7043-D_TANTALUM-220UF" value="220uF"/>
+<part name="C25" library="quadparts_prebuilt" deviceset="CAPACITOR-POL_" device="SMD-7043-D_TANTALUM-220UF" value="220uF"/>
+<part name="GND15" library="quadparts_prebuilt" deviceset="BAT_GND" device=""/>
+<part name="GND21" library="quadparts_prebuilt" deviceset="BAT_GND" device=""/>
+<part name="GND24" library="quadparts_prebuilt" deviceset="BAT_GND" device=""/>
+<part name="GND26" library="quadparts_prebuilt" deviceset="BAT_GND" device=""/>
 </parts>
 <sheets>
@@
 <instance part="D4" gate="G$1" x="-995.68" y="1104.9" rot="R90"/>
 <instance part="C18" gate="G$1" x="-1389.38" y="1097.28"/>
+<instance part="C7" gate="G$1" x="-1198.88" y="1104.9"/>
+<instance part="C8" gate="G$1" x="-1122.68" y="1104.9"/>
+<instance part="C24" gate="G$1" x="-1049.02" y="1104.9"/>
+<instance part="C25" gate="G$1" x="-977.9" y="1104.9"/>
+<instance part="GND15" gate="1" x="-977.9" y="1092.2"/>
+<instance part="GND21" gate="1" x="-1049.02" y="1092.2"/>
+<instance part="GND24" gate="1" x="-1198.88" y="1092.2"/>
+<instance part="GND26" gate="1" x="-1122.68" y="1092.2"/>
 </instances>
 <busses>
@@
 <junction x="-1008.38" y="1107.44"/>
 <wire x1="-995.68" y1="1109.98" x2="-995.68" y2="1122.68" width="0.1524" layer="91"/>
-<wire x1="-995.68" y1="1122.68" x2="-1069.34" y2="1122.68" width="0.1524" layer="91"/>
+<wire x1="-995.68" y1="1122.68" x2="-1005.84" y2="1122.68" width="0.1524" layer="91"/>
 <pinref part="U$3" gate="G$1" pin="V+"/>
+<wire x1="-1005.84" y1="1122.68" x2="-1049.02" y2="1122.68" width="0.1524" layer="91"/>
+<wire x1="-1049.02" y1="1122.68" x2="-1069.34" y2="1122.68" width="0.1524" layer="91"/>
 <wire x1="-1082.04" y1="1107.44" x2="-1082.04" y2="1109.98" width="0.1524" layer="91"/>
 <wire x1="-1082.04" y1="1109.98" x2="-1069.34" y2="1109.98" width="0.1524" layer="91"/>
 <wire x1="-1069.34" y1="1107.44" x2="-1069.34" y2="1109.98" width="0.1524" layer="91"/>
 <junction x="-1082.04" y="1107.44"/>
-<wire x1="-1143" y1="1122.68" x2="-1069.34" y2="1122.68" width="0.1524" layer="91"/>
+<wire x1="-1143" y1="1122.68" x2="-1122.68" y2="1122.68" width="0.1524" layer="91"/>
+<wire x1="-1122.68" y1="1122.68" x2="-1069.34" y2="1122.68" width="0.1524" layer="91"/>
 <wire x1="-1069.34" y1="1122.68" x2="-1069.34" y2="1109.98" width="0.1524" layer="91"/>
 <wire x1="-1143" y1="1109.98" x2="-1143" y2="1122.68" width="0.1524" layer="91"/>
@@
 <wire x1="-1216.66" y1="1107.44" x2="-1216.66" y2="1109.98" width="0.1524" layer="91"/>
 <junction x="-1229.36" y="1107.44"/>
-<wire x1="-1143" y1="1122.68" x2="-1216.66" y2="1122.68" width="0.1524" layer="91"/>
+<wire x1="-1143" y1="1122.68" x2="-1198.88" y2="1122.68" width="0.1524" layer="91"/>
+<wire x1="-1198.88" y1="1122.68" x2="-1216.66" y2="1122.68" width="0.1524" layer="91"/>
 <wire x1="-1216.66" y1="1109.98" x2="-1216.66" y2="1122.68" width="0.1524" layer="91"/>
 <wire x1="-1216.66" y1="1122.68" x2="-1244.6" y2="1122.68" width="0.1524" layer="91"/>
@@
 <junction x="-995.68" y="1107.44"/>
 <junction x="-1216.66" y="1107.44"/>
+<junction x="-1069.34" y="1122.68"/>
+<pinref part="C24" gate="G$1" pin="+"/>
+<wire x1="-1049.02" y1="1107.44" x2="-1049.02" y2="1122.68" width="0.1524" layer="91"/>
+<pinref part="C8" gate="G$1" pin="+"/>
+<wire x1="-1122.68" y1="1107.44" x2="-1122.68" y2="1122.68" width="0.1524" layer="91"/>
+<wire x1="-1198.88" y1="1104.9" x2="-1198.88" y2="1107.44" width="0.1524" layer="91"/>
+<pinref part="C25" gate="G$1" pin="+"/>
+<wire x1="-1198.88" y1="1107.44" x2="-1198.88" y2="1122.68" width="0.1524" layer="91"/>
+<wire x1="-977.9" y1="1107.44" x2="-977.9" y2="1122.68" width="0.1524" layer="91"/>
+<wire x1="-977.9" y1="1122.68" x2="-995.68" y2="1122.68" width="0.1524" layer="91"/>
+<pinref part="C7" gate="G$1" pin="+"/>
+<junction x="-1198.88" y="1107.44"/>
+<junction x="-1198.88" y="1122.68"/>
+<junction x="-1122.68" y="1107.44"/>
+<junction x="-1122.68" y="1122.68"/>
+<junction x="-1049.02" y="1107.44"/>
+<junction x="-1049.02" y="1122.68"/>
+<junction x="-995.68" y="1122.68"/>
+<junction x="-977.9" y="1122.68"/>
+<junction x="-977.9" y="1107.44"/>
 </segment>
 <segment>
@@
 <junction x="-1010.92" y="1033.78"/>
 </segment>
-</net>
+<segment>
+<pinref part="C25" gate="G$1" pin="-"/>
+<wire x1="-977.9" y1="1099.82" x2="-977.9" y2="1094.74" width="0.1524" layer="91"/>
+<pinref part="GND15" gate="1" pin="BAT_GND"/>
+<junction x="-977.9" y="1094.74"/>
+<junction x="-977.9" y="1099.82"/>
+</segment>
+<segment>
+<pinref part="C24" gate="G$1" pin="-"/>
+<wire x1="-1049.02" y1="1099.82" x2="-1049.02" y2="1094.74" width="0.1524" layer="91"/>
+<pinref part="GND21" gate="1" pin="BAT_GND"/>
+<junction x="-1049.02" y="1094.74"/>
+<junction x="-1049.02" y="1099.82"/>
+</segment>
+<segment>
+<pinref part="C7" gate="G$1" pin="-"/>
+<wire x1="-1198.88" y1="1099.82" x2="-1198.88" y2="1094.74" width="0.1524" layer="91"/>
+<pinref part="GND24" gate="1" pin="BAT_GND"/>
+<junction x="-1198.88" y="1094.74"/>
+<junction x="-1198.88" y="1099.82"/>
+</segment>
+<segment>
+<pinref part="C8" gate="G$1" pin="-"/>
+<wire x1="-1122.68" y1="1099.82" x2="-1122.68" y2="1094.74" width="0.1524" layer="91"/>
+<pinref part="GND26" gate="1" pin="BAT_GND"/>
+<junction x="-1122.68" y="1099.82"/>
+<junction x="-1122.68" y="1094.74"/>
+</segment>
+</net>
