File: quadcopter.brd (EAGLE design)
At the start: 134.1 x 134 mm, 81 parts, among them J1 ISP, U2 ATMEGA128RFA1

Commit message: After fixing professor's comments V4 (GND)
Parts:
- moved C23 8.99 mm to (-5.23, -36.1)
Routing:
- net GND: track 205.3 -> 214.0 mm, vias 11 -> 29
- net DVDD: track 8.25 -> 16.9 mm
- added copper zone on layer 1, net GND
- added copper zone on layer 16, net GND
- added copper zone on layer 2, net GND

Commit message: After fixing professor's comments V4 (GND)
Parts:
- moved C9 5.88 mm to (-22.7, -25.6), turned to 270 degrees
- moved C22 0.81 mm to (-20.6, -25.5)
- turned C11 to 270 degrees
Routing:
- net GND: track 214.0 -> 208.2 mm
- net AVDD: track 5.86 -> 7.67 mm
- net RFANT: track 8.06 -> 6.46 mm
- net VBAT_SENSE: track 11.9 -> 12.7 mm
Other:
- board text added: "HKN TEAM: ANDREW S. LUCAS T."
